Commit message: Update package file names. TODO programmatic way

File: lk_rmc_description/urdf/model.xacro (robot description, xacro)
@@ -28,19 +28,19 @@
       <geometry>
         <mesh
-          filename="package://lk_description/meshes/base_link.STL" />
-      </geometry>
-      <material
-        name="">
-        <color
-          rgba="0.79216 0.81961 0.93333 1" />
-      </material>
-    </visual>
-    <collision>
-      <origin
-        xyz="0 0 0"
-        rpy="0 0 0" />
-      <geometry>
-        <mesh
-          filename="package://lk_description/meshes/base_link.STL" />
+          filename="package://lk_rmc_description/meshes/base_link.STL" />
+      </geometry>
+      <material
+        name="">
+        <color
+          rgba="0.79216 0.81961 0.93333 1" />
+      </material>
+    </visual>
+    <collision>
+      <origin
+        xyz="0 0 0"
+        rpy="0 0 0" />
+      <geometry>
+        <mesh
+          filename="package://lk_rmc_description/meshes/base_link.STL" />
       </geometry>
     </collision>
@@ -69,19 +69,19 @@
           <cylinder length=".1016" radius=".1524"/>
         <!-- <mesh
-          filename="package://lk_description/meshes/frontLeftWheel.STL" /> -->
-      </geometry>
-      <material
-        name="">
-        <color
-          rgba="0.79216 0.81961 0.93333 1" />
-      </material>
-    </visual>
-    <collision>
-      <origin
-        xyz="0 0 0"
-        rpy="0 0 0" />
-      <geometry>
-        <!-- <mesh
-          filename="package://lk_description/meshes/frontLeftWheel.STL" /> -->
+          filename="package://lk_rmc_description/meshes/frontLeftWheel.STL" /> -->
+      </geometry>
+      <material
+        name="">
+        <color
+          rgba="0.79216 0.81961 0.93333 1" />
+      </material>
+    </visual>
+    <collision>
+      <origin
+        xyz="0 0 0"
+        rpy="0 0 0" />
+      <geometry>
+        <!-- <mesh
+          filename="package://lk_rmc_description/meshes/frontLeftWheel.STL" /> -->
         <cylinder length=".1016" radius=".1524"/>
       </geometry>
@@ -123,5 +123,5 @@
       <geometry>
         <!-- <mesh
-          filename="package://lk_description/meshes/backLeftWheel.STL" /> -->
+          filename="package://lk_rmc_description/meshes/backLeftWheel.STL" /> -->
                   <cylinder length=".1016" radius=".1524"/>
       </geometry>
@@ -138,5 +138,5 @@
       <geometry>
         <!-- <mesh
-          filename="package://lk_description/meshes/backLeftWheel.STL" /> -->
+          filename="package://lk_rmc_description/meshes/backLeftWheel.STL" /> -->
                   <cylinder length=".1016" radius=".1524"/>
       </geometry>
@@ -178,5 +178,5 @@
       <geometry>
         <!-- <mesh
-          filename="package://lk_description/meshes/frontRightWheel.STL" /> -->
+          filename="package://lk_rmc_description/meshes/frontRightWheel.STL" /> -->
                   <cylinder length=".1016" radius=".1524"/>
       </geometry>
@@ -193,5 +193,5 @@
       <geometry>
         <!-- <mesh
-          filename="package://lk_description/meshes/frontRightWheel.STL" /> -->
+          filename="package://lk_rmc_description/meshes/frontRightWheel.STL" /> -->
                   <cylinder length=".1016" radius=".1524"/>
       </geometry>
@@ -233,5 +233,5 @@
       <geometry>
         <!-- <mesh
-          filename="package://lk_description/meshes/backRightWheel.STL" /> -->
+          filename="package://lk_rmc_description/meshes/backRightWheel.STL" /> -->
                   <cylinder length=".1016" radius=".1524"/>
       </geometry>
@@ -248,5 +248,5 @@
       <geometry>
         <!-- <mesh
-          filename="package://lk_description/meshes/backRightWheel.STL" /> -->
+          filename="package://lk_rmc_description/meshes/backRightWheel.STL" /> -->
                   <cylinder length=".1016" radius=".1524"/>
       </geometry>
@@ -288,19 +288,19 @@
       <geometry>
         <mesh
-          filename="package://lk_description/meshes/depRightActuator.STL" />
-      </geometry>
-      <material
-        name="">
-        <color
-          rgba="0.79216 0.81961 0.93333 1" />
-      </material>
-    </visual>
-    <collision>
-      <origin
-        xyz="0 0 0"
-        rpy="0 0 0" />
-      <geometry>
-        <mesh
-          filename="package://lk_description/meshes/depRightActuator.STL" />
+          filename="package://lk_rmc_description/meshes/depRightActuator.STL" />
+      </geometry>
+      <material
+        name="">
+        <color
+          rgba="0.79216 0.81961 0.93333 1" />
+      </material>
+    </visual>
+    <collision>
+      <origin
+        xyz="0 0 0"
+        rpy="0 0 0" />
+      <geometry>
+        <mesh
+          filename="package://lk_rmc_description/meshes/depRightActuator.STL" />
       </geometry>
     </collision>
@@ -344,19 +344,19 @@
       <geometry>
         <mesh
-          filename="package://lk_description/meshes/depConveyor.STL" />
-      </geometry>
-      <material
-        name="">
-        <color
-          rgba="0.79216 0.81961 0.93333 1" />
-      </material>
-    </visual>
-    <collision>
-      <origin
-        xyz="0 0 0"
-        rpy="0 0 0" />
-      <geometry>
-        <mesh
-          filename="package://lk_description/meshes/depConveyor.STL" />
+          filename="package://lk_rmc_description/meshes/depConveyor.STL" />
+      </geometry>
+      <material
+        name="">
+        <color
+          rgba="0.79216 0.81961 0.93333 1" />
+      </material>
+    </visual>
+    <collision>
+      <origin
+        xyz="0 0 0"
+        rpy="0 0 0" />
+      <geometry>
+        <mesh
+          filename="package://lk_rmc_description/meshes/depConveyor.STL" />
       </geometry>
     </collision>
@@ -397,19 +397,19 @@
       <geometry>
         <mesh
-          filename="package://lk_description/meshes/depLeftActuator.STL" />
-      </geometry>
-      <material
-        name="">
-        <color
-          rgba="0.79216 0.81961 0.93333 1" />
-      </material>
-    </visual>
-    <collision>
-      <origin
-        xyz="0 0 0"
-        rpy="0 0 0" />
-      <geometry>
-        <mesh
-          filename="package://lk_description/meshes/depLeftActuator.STL" />
+          filename="package://lk_rmc_description/meshes/depLeftActuator.STL" />
+      </geometry>
+      <material
+        name="">
+        <color
+          rgba="0.79216 0.81961 0.93333 1" />
+      </material>
+    </visual>
+    <collision>
+      <origin
+        xyz="0 0 0"
+        rpy="0 0 0" />
+      <geometry>
+        <mesh
+          filename="package://lk_rmc_description/meshes/depLeftActuator.STL" />
       </geometry>
     </collision>
@@ -453,5 +453,5 @@
       <geometry>
         <mesh
-          filename="package://lk_description/meshes/cameraActuator.STL" />
+          filename="package://lk_rmc_description/meshes/cameraActuator.STL" />
       </geometry>
       <material
@@ -467,5 +467,5 @@
       <geometry>
         <mesh
-          filename="package://lk_description/meshes/cameraActuator.STL" />
+          filename="package://lk_rmc_description/meshes/cameraActuator.STL" />
       </geometry>
     </collision>
@@ -509,19 +509,19 @@
       <geometry>
         <mesh
-          filename="package://lk_description/meshes/intakeConveyor.STL" />
-      </geometry>
-      <material
-        name="">
-        <color
-          rgba="0.79216 0.81961 0.93333 1" />
-      </material>
-    </visual>
-    <collision>
-      <origin
-        xyz="0 0 0"
-        rpy="0 0 0" />
-      <geometry>
-        <mesh
-          filename="package://lk_description/meshes/intakeConveyor.STL" />
+          filename="package://lk_rmc_description/meshes/intakeConveyor.STL" />
+      </geometry>
+      <material
+        name="">
+        <color
+          rgba="0.79216 0.81961 0.93333 1" />
+      </material>
+    </visual>
+    <collision>
+      <origin
+        xyz="0 0 0"
+        rpy="0 0 0" />
+      <geometry>
+        <mesh
+          filename="package://lk_rmc_description/meshes/intakeConveyor.STL" />
       </geometry>
     </collision>

Commit message: Added files. Rviz looks correct, gazebo doesnt

File: lk_rmc_description/urdf/model.xacro (robot description, xacro)
@@ -1,9 +1,10 @@
 <robot
   name="sirdigsalot">
-  <!-- <link name="world"/> -->
-  <!-- <joint name="fixed" type="fixed">
-    <parent link="world"/>
+  <link name="base_footprint"/>
+  <joint name="base_joint" type="fixed">
+    <parent link = "base_footprint"/>
     <child link="base_link"/>
-  </joint> -->
+    <origin xyz="0.0 0.0 0.5" rpy="0 0 0 "/>
+  </joint>
   <link
     name="base_link">
@@ -13,11 +14,11 @@
         rpy="0 0 0" />
       <mass
-        value="12.883" />
+        value="2.0" />
       <inertia
         ixx="0.27816"
         ixy="-0.020687"
-        ixz="1.9963E-05"
+        ixz="0"
         iyy="0.59209"
-        iyz="3.0096E-05"
+        iyz="0"
         izz="0.60601" />
     </inertial>
@@ -53,5 +54,5 @@
         rpy="0 0 0" />
       <mass
-        value="7.4005" />
+        value="1.0" />
       <inertia
         ixx="0"
@@ -68,6 +69,4 @@
       <geometry>
           <cylinder length=".1016" radius=".1524"/>
-        <!-- <mesh
-          filename="package://lk_rmc_description/meshes/frontLeftWheel.STL" /> -->
       </geometry>
       <material
@@ -82,6 +81,4 @@
         rpy="0 0 0" />
       <geometry>
-        <!-- <mesh
-          filename="package://lk_rmc_description/meshes/frontLeftWheel.STL" /> -->
         <cylinder length=".1016" radius=".1524"/>
       </geometry>
@@ -108,5 +105,5 @@
         rpy="0 0 0" />
       <mass
-        value="7.4005" />
+        value="1.0" />
       <inertia
         ixx="0"
@@ -122,7 +119,5 @@
         rpy="0 0 0" />
       <geometry>
-        <!-- <mesh
-          filename="package://lk_rmc_description/meshes/backLeftWheel.STL" /> -->
-                  <cylinder length=".1016" radius=".1524"/>
+        <cylinder length=".1016" radius=".1524"/>
       </geometry>
       <material
@@ -137,7 +132,5 @@
         rpy="0 0 0" />
       <geometry>
-        <!-- <mesh
-          filename="package://lk_rmc_description/meshes/backLeftWheel.STL" /> -->
-                  <cylinder length=".1016" radius=".1524"/>
+        <cylinder length=".1016" radius=".1524"/>
       </geometry>
     </collision>
@@ -163,5 +156,5 @@
         rpy="0 0 0" />
       <mass
-        value="7.4005" />
+        value="1.0" />
       <inertia
         ixx="0"
@@ -177,7 +170,5 @@
         rpy="0 0 0" />
       <geometry>
-        <!-- <mesh
-          filename="package://lk_rmc_description/meshes/frontRightWheel.STL" /> -->
-                  <cylinder length=".1016" radius=".1524"/>
+        <cylinder length=".1016" radius=".1524"/>
       </geometry>
       <material
@@ -192,7 +183,5 @@
         rpy="0 0 0" />
       <geometry>
-        <!-- <mesh
-          filename="package://lk_rmc_description/meshes/frontRightWheel.STL" /> -->
-                  <cylinder length=".1016" radius=".1524"/>
+        <cylinder length=".1016" radius=".1524"/>
       </geometry>
     </collision>
@@ -211,46 +200,4 @@
       xyz="0 0 1" />
   </joint>
-  <link
-    name="backRightWheel">
-    <inertial>
-      <origin
-        xyz="5.55111512312578E-17 0 0.0508"
-        rpy="0 0 0" />
-      <mass
-        value="7.40046273221895" />
-      <inertia
-        ixx="0"
-        ixy="0"
-        ixz="0"
-        iyy="0"
-        iyz="0"
-        izz="0" />
-    </inertial>
-    <visual>
-      <origin
-        xyz="0 0 0"
-        rpy="0 0 0" />
-      <geometry>
-        <!-- <mesh
-          filename="package://lk_rmc_description/meshes/backRightWheel.STL" /> -->
-                  <cylinder length=".1016" radius=".1524"/>
-      </geometry>
-      <material
-        name="">
-        <color
-          rgba="0.792156862745098 0.819607843137255 0.933333333333333 1" />
-      </material>
-    </visual>
-    <collision>
-      <origin
-        xyz="0 0 0"
-        rpy="0 0 0" />
-      <geometry>
-        <!-- <mesh
-          filename="package://lk_rmc_description/meshes/backRightWheel.STL" /> -->
-                  <cylinder length=".1016" radius=".1524"/>
-      </geometry>
-    </collision>
-  </link>
   <joint
     name="backRightWheelRotate"
@@ -266,12 +213,12 @@
       xyz="0 0 1" />
   </joint>
-  <!-- <link
-    name="depRightActuator">
-    <inertial>
-      <origin
-        xyz="-4.2562E-09 -0.020725 3.5813E-09"
-        rpy="0 0 0" />
-      <mass
-        value="0.088669" />
+  <link
+    name="backRightWheel">
+    <inertial>
+      <origin
+        xyz="0 0 0.0"
+        rpy="0 0 0" />
+      <mass
+        value="1.0" />
       <inertia
         ixx="0"
@@ -287,308 +234,67 @@
         rpy="0 0 0" />
       <geometry>
-        <mesh
-          filename="package://lk_rmc_description/meshes/depRightActuator.STL" />
-      </geometry>
-      <material
-        name="">
-        <color
-          rgba="0.79216 0.81961 0.93333 1" />
-      </material>
-    </visual>
-    <collision>
-      <origin
-        xyz="0 0 0"
-        rpy="0 0 0" />
-      <geometry>
-        <mesh
-          filename="package://lk_rmc_description/meshes/depRightActuator.STL" />
-      </geometry>
-    </collision>
-  </link> -->
-  <!-- <joint
-    name="depRightExtend"
-    type="prismatic">
-    <origin
-      xyz="-0.11281 -0.18528 0"
-      rpy="-1.5708 0 0" />
-    <parent
-      link="base_link" />
-    <child
-      link="depRightActuator" />
-    <axis
-      xyz="0 -1 0" />
-    <limit
-      effort="0"
-      velocity="0" />
-  </joint>
-  <link
-    name="depConveyor">
-    <inertial>
-      <origin
-        xyz="0.28997 -6.0219E-05 0.15395"
-        rpy="0 0 0" />
-      <mass
-        value="22.501" />
-      <inertia
-        ixx="0.039859"
-        ixy="6.0953E-06"
-        ixz="0.047728"
-        iyy="0.097009"
-        iyz="-5.0904E-06"
-        izz="0.05715" />
-    </inertial>
-    <visual>
-      <origin
-        xyz="0 0 0"
-        rpy="0 0 0" />
-      <geometry>
-        <mesh
-          filename="package://lk_rmc_description/meshes/depConveyor.STL" />
-      </geometry>
-      <material
-        name="">
-        <color
-          rgba="0.79216 0.81961 0.93333 1" />
-      </material>
-    </visual>
-    <collision>
-      <origin
-        xyz="0 0 0"
-        rpy="0 0 0" />
-      <geometry>
-        <mesh
-          filename="package://lk_rmc_description/meshes/depConveyor.STL" />
-      </geometry>
-    </collision>
-  </link>
-  <joint
-    name="depConveyorRotate"
-    type="fixed">
-    <origin
-      xyz="-0.36547 -0.16157 0.32661"
-      rpy="3.1416 0 0.48826" />
-    <parent
-      link="depRightActuator" />
-    <child
-      link="depConveyor" />
-    <axis
-      xyz="0 0 0" />
-  </joint>
-  <link
-    name="depLeftActuator">
-    <inertial>
-      <origin
-        xyz="-4.2562E-09 -0.020725 3.5813E-09"
-        rpy="0 0 0" />
-      <mass
-        value="0.088669" />
-      <inertia
-        ixx="0"
-        ixy="0"
-        ixz="0"
-        iyy="0"
-        iyz="0"
-        izz="0" />
-    </inertial>
-    <visual>
-      <origin
-        xyz="0 0 0"
-        rpy="0 0 0" />
-      <geometry>
-        <mesh
-          filename="package://lk_rmc_description/meshes/depLeftActuator.STL" />
-      </geometry>
-      <material
-        name="">
-        <color
-          rgba="0.79216 0.81961 0.93333 1" />
-      </material>
-    </visual>
-    <collision>
-      <origin
-        xyz="0 0 0"
-        rpy="0 0 0" />
-      <geometry>
-        <mesh
-          filename="package://lk_rmc_description/meshes/depLeftActuator.STL" />
-      </geometry>
-    </collision>
-  </link>
-  <joint
-    name="depLeftExtend"
-    type="prismatic">
-    <origin
-      xyz="-0.11281 0.1815 0"
-      rpy="-1.5708 6.3639E-19 3.1312" />
-    <parent
-      link="base_link" />
-    <child
-      link="depLeftActuator" />
-    <axis
-      xyz="0 -1 0" />
-    <limit
-      effort="0"
-      velocity="0" />
-  </joint>
-  <link
-    name="cameraActuator">
-    <inertial>
-      <origin
-        xyz="-2.73470979195167E-09 0.124252406834887 -1.03760512334961E-09"
-        rpy="0 0 0" />
-      <mass
-        value="0.210658735046211" />
-      <inertia
-        ixx="0"
-        ixy="0"
-        ixz="0"
-        iyy="0"
-        iyz="0"
-        izz="0" />
-    </inertial>
-    <visual>
-      <origin
-        xyz="0 0 0"
-        rpy="0 0 0" />
-      <geometry>
-        <mesh
-          filename="package://lk_rmc_description/meshes/cameraActuator.STL" />
-      </geometry>
-      <material
-        name="">
-        <color
-          rgba="0.898039215686275 0.917647058823529 0.929411764705882 1" />
-      </material>
-    </visual>
-    <collision>
-      <origin
-        xyz="0 0 0"
-        rpy="0 0 0" />
-      <geometry>
-        <mesh
-          filename="package://lk_rmc_description/meshes/cameraActuator.STL" />
-      </geometry>
-    </collision>
-  </link>
-  <joint
-    name="cameraExtend"
-    type="prismatic">
-    <origin
-      xyz="0.41957 -0.0018055 0.0051623"
-      rpy="1.5708 -3.9284E-18 -0.064201" />
-    <parent
-      link="base_link" />
-    <child
-      link="cameraActuator" />
-    <axis
-      xyz="0 1 0" />
-    <limit
-      effort="0"
-      velocity="0" />
-  </joint>
-  <link
-    name="intakeConveyor">
-    <inertial>
-      <origin
-        xyz="-3.0286E-08 -0.0087509 0.085493"
-        rpy="0 0 0" />
-      <mass
-        value="31.448" />
-      <inertia
-        ixx="0"
-        ixy="0"
-        ixz="0"
-        iyy="0"
-        iyz="0"
-        izz="0" />
-    </inertial>
-    <visual>
-      <origin
-        xyz="0 0 0"
-        rpy="0 0 0" />
-      <geometry>
-        <mesh
-          filename="package://lk_rmc_description/meshes/intakeConveyor.STL" />
-      </geometry>
-      <material
-        name="">
-        <color
-          rgba="0.79216 0.81961 0.93333 1" />
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
Commit message: Fix some inertial properties. Working Gazebo

File: lk_rmc_description/urdf/model.xacro (robot description, xacro)
@@ -9,18 +9,4 @@
   <link
     name="base_link">
-    <inertial>
-      <origin
-        xyz="0.0063713 -0.11708 0.0018811"
-        rpy="0 0 0" />
-      <mass
-        value="2.0" />
-      <inertia
-        ixx="0.27816"
-        ixy="-0.020687"
-        ixz="0"
-        iyy="0.59209"
-        iyz="0"
-        izz="0.60601" />
-    </inertial>
     <visual>
       <origin
@@ -46,21 +32,15 @@
       </geometry>
     </collision>
+    <inertial>
+      <origin xyz="0 0 -.25" rpy="0 0 0"/>
+      <mass value="12"/>
+      <inertia
+        ixx="1.0" ixy="0.0" ixz="0.0"
+        iyy="1.0" iyz="0.0"
+        izz="1.0"/>
+    </inertial>
   </link>
   <link
     name="frontLeftWheel">
-    <inertial>
-      <origin
-        xyz="0 0 -0.0508"
-        rpy="0 0 0" />
-      <mass
-        value="1.0" />
-      <inertia
-        ixx="0"
-        ixy="0"
-        ixz="0"
-        iyy="0"
-        iyz="0"
-        izz="0" />
-    </inertial>
     <visual>
       <origin
@@ -84,4 +64,12 @@
       </geometry>
     </collision>
+    <inertial>
+      <origin xyz="0 0 0" rpy="0 0 0"/>
+      <mass value="5"/>
+      <inertia
+        ixx="1.0" ixy="0.0" ixz="0.0"
+        iyy="1.0" iyz="0.0"
+        izz="1.0"/>
+    </inertial>
   </link>
   <joint
@@ -100,39 +88,33 @@
   <link
     name="backLeftWheel">
-    <inertial>
-      <origin
-        xyz="-1.6653E-16 -1.9602E-16 -0.0508"
-        rpy="0 0 0" />
-      <mass
-        value="1.0" />
-      <inertia
-        ixx="0"
-        ixy="0"
-        ixz="0"
-        iyy="0"
-        iyz="0"
-        izz="0" />
-    </inertial>
-    <visual>
-      <origin
-        xyz="0 0 0"
-        rpy="0 0 0" />
-      <geometry>
-        <cylinder length=".1016" radius=".1524"/>
-      </geometry>
-      <material
-        name="">
-        <color
-          rgba="0.79216 0.81961 0.93333 1" />
-      </material>
-    </visual>
-    <collision>
-      <origin
-        xyz="0 0 0"
-        rpy="0 0 0" />
-      <geometry>
-        <cylinder length=".1016" radius=".1524"/>
-      </geometry>
-    </collision>
+    <visual>
+      <origin
+        xyz="0 0 0"
+        rpy="0 0 0" />
+      <geometry>
+        <cylinder length=".1016" radius=".1524"/>
+      </geometry>
+      <material
+        name="">
+        <color
+          rgba="0.79216 0.81961 0.93333 1" />
+      </material>
+    </visual>
+    <collision>
+      <origin
+        xyz="0 0 0"
+        rpy="0 0 0" />
+      <geometry>
+        <cylinder length=".1016" radius=".1524"/>
+      </geometry>
+    </collision>
+    <inertial>
+      <origin xyz="0 0 0" rpy="0 0 0"/>
+      <mass value="5"/>
+      <inertia
+        ixx="1.0" ixy="0.0" ixz="0.0"
+        iyy="1.0" iyz="0.0"
+        izz="1.0"/>
+    </inertial>
   </link>
   <joint
@@ -151,39 +133,33 @@
   <link
     name="frontRightWheel">
-    <inertial>
-      <origin
-        xyz="0 0 0.0508"
-        rpy="0 0 0" />
-      <mass
-        value="1.0" />
-      <inertia
-        ixx="0"
-        ixy="0"
-        ixz="0"
-        iyy="0"
-        iyz="0"
-        izz="0" />
-    </inertial>
-    <visual>
-      <origin
-        xyz="0 0 0"
-        rpy="0 0 0" />
-      <geometry>
-        <cylinder length=".1016" radius=".1524"/>
-      </geometry>
-      <material
-        name="">
-        <color
-          rgba="0.79216 0.81961 0.93333 1" />
-      </material>
-    </visual>
-    <collision>
-      <origin
-        xyz="0 0 0"
-        rpy="0 0 0" />
-      <geometry>
-        <cylinder length=".1016" radius=".1524"/>
-      </geometry>
-    </collision>
+    <visual>
+      <origin
+        xyz="0 0 0"
+        rpy="0 0 0" />
+      <geometry>
+        <cylinder length=".1016" radius=".1524"/>
+      </geometry>
+      <material
+        name="">
+        <color
+          rgba="0.79216 0.81961 0.93333 1" />
+      </material>
+    </visual>
+    <collision>
+      <origin
+        xyz="0 0 0"
+        rpy="0 0 0" />
+      <geometry>
+        <cylinder length=".1016" radius=".1524"/>
+      </geometry>
+    </collision>
+    <inertial>
+      <origin xyz="0 0 0" rpy="0 0 0"/>
+      <mass value="5"/>
+      <inertia
+        ixx="1.0" ixy="0.0" ixz="0.0"
+        iyy="1.0" iyz="0.0"
+        izz="1.0"/>
+    </inertial>
   </link>
   <joint
@@ -215,18 +191,4 @@
   <link
     name="backRightWheel">
-    <inertial>
-      <origin
-        xyz="0 0 0.0"
-        rpy="0 0 0" />
-      <mass
-        value="1.0" />
-      <inertia
-        ixx="0"
-        ixy="0"
-        ixz="0"
-        iyy="0"
-        iyz="0"
-        izz="0" />
-    </inertial>
     <visual>
       <origin
@@ -250,4 +212,12 @@
       </geometry>
     </collision>
+    <inertial>
+      <origin xyz="0 0 0" rpy="0 0 0"/>
+      <mass value="5"/>
+      <inertia
+        ixx="1.0" ixy="0.0" ixz="0.0"
+        iyy="1.0" iyz="0.0"
+        izz="1.0"/>
+    </inertial>
   </link>
   <gazebo>
