Commit message: Add IMU & stereo sensor inputs from gazebo

File: lk_rmc_description/urdf/model.xacro (robot description, xacro)
@@ -5,5 +5,5 @@
     <parent link = "base_footprint"/>
     <child link="base_link"/>
-    <origin xyz="0.0 0.0 0.5" rpy="0 0 0 "/>
+    <origin xyz="0.0 0.0 0.4" rpy="0 0 0 "/>
   </joint>
   <link
@@ -221,4 +221,16 @@
     </inertial>
   </link>
+  <link name="imu_link"/>
+  <joint name="imu_joint" type="fixed">
+    <parent link = "base_link"/>
+    <child link="imu_link"/>
+    <origin xyz="0.0 0.0 0.0" rpy="0 0 0 "/>
+  </joint>
+  <link name="left_camera_frame"/>
+  <joint name="left_camera_frame" type="fixed">
+    <parent link = "base_link"/>
+    <child link="left_camera_frame"/>
+    <origin xyz="0.0 0.0 0.0" rpy="0 0 0 "/>
+  </joint>
   <gazebo>
     <plugin name="gazebo_ros_control" filename="libgazebo_ros_control.so">
@@ -268,3 +280,77 @@
     </joint>
   </transmission>
+  <gazebo reference="imu_link">
+    <gravity>true</gravity>
+    <sensor name="imu_sensor" type="imu">
+      <always_on>true</always_on>
+      <update_rate>100</update_rate>
+      <visualize>true</visualize>
+      <topic>__default_topic__</topic>
+      <plugin filename="libgazebo_ros_imu_sensor.so" name="imu_plugin">
+        <topicName>imu</topicName>
+        <bodyName>imu_link</bodyName>
+        <updateRateHZ>10.0</updateRateHZ>
+        <gaussianNoise>0.0</gaussianNoise>
+        <xyzOffset>0 0 0</xyzOffset>
+        <rpyOffset>0 0 0</rpyOffset>
+        <frameName>imu_link</frameName>
+      </plugin>
+      <pose>0 0 0 0 0 0</pose>
+    </sensor>
+  </gazebo>
+  <gazebo reference="left_camera_frame">
+    <sensor type="multicamera" name="stereo_camera">
+      <update_rate>30.0</update_rate>
+      <camera name="left">
+        <horizontal_fov>1.3962634</horizontal_fov>
+        <image>
+          <width>800</width>
+          <height>800</height>
+          <format>R8G8B8</format>
+        </image>
+        <clip>
+          <near>0.02</near>
+          <far>300</far>
+        </clip>
+        <noise>
+          <type>gaussian</type>
+          <mean>0.0</mean>
+          <stddev>0.007</stddev>
+        </noise>
+      </camera>
+      <camera name="right">
+        <pose>0 -0.07 0 0 0 0</pose>
+        <horizontal_fov>1.3962634</horizontal_fov>
+        <image>
+          <width>800</width>
+          <height>800</height>
+          <format>R8G8B8</format>
+        </image>
+        <clip>
+          <near>0.02</near>
+          <far>300</far>
+        </clip>
+        <noise>
+          <type>gaussian</type>
+          <mean>0.0</mean>
+          <stddev>0.007</stddev>
+        </noise>
+      </camera>
+      <plugin name="stereo_camera_controller" filename="libgazebo_ros_multicamera.so">
+        <alwaysOn>true</alwaysOn>
+        <updateRate>0.0</updateRate>
+        <cameraName>multisense_sl/camera</cameraName>
+        <imageTopicName>image_raw</imageTopicName>
+        <cameraInfoTopicName>camera_info</cameraInfoTopicName>
+        <frameName>left_camera_optical_frame</frameName>
+        <!--<rightFrameName>right_camera_optical_frame</rightFrameName>-->
+        <hackBaseline>0.07</hackBaseline>
+        <distortionK1>0.0</distortionK1>
+        <distortionK2>0.0</distortionK2>
+        <distortionK3>0.0</distortionK3>
+        <distortionT1>0.0</distortionT1>
+        <distortionT2>0.0</distortionT2>
+      </plugin>
+    </sensor>
+  </gazebo>
 </robot>

Commit message: Added sensors and adjusted links to urdf

File: lk_rmc_description/urdf/model.xacro (robot description, xacro)
@@ -227,9 +227,15 @@
     <origin xyz="0.0 0.0 0.0" rpy="0 0 0 "/>
   </joint>
-  <link name="left_camera_frame"/>
-  <joint name="left_camera_frame" type="fixed">
+  <link name="camera_link"/>
+  <joint name="camera_link" type="fixed">
     <parent link = "base_link"/>
-    <child link="left_camera_frame"/>
-    <origin xyz="0.0 0.0 0.0" rpy="0 0 0 "/>
+    <child link="camera_link"/>
+    <origin xyz="0.385 0.0 0.235" rpy="0 0 0 "/>
+  </joint>
+  <link name="laser_link"/>
+  <joint name="laser_link" type="fixed">
+    <parent link = "base_link"/>
+    <child link="laser_link"/>
+    <origin xyz="0.385 0.0 0.235" rpy="0 0 0 "/>
   </joint>
   <gazebo>
@@ -299,5 +305,5 @@
     </sensor>
   </gazebo>
-  <gazebo reference="left_camera_frame">
+  <gazebo reference="camera_link">
     <sensor type="multicamera" name="stereo_camera">
       <update_rate>30.0</update_rate>
@@ -354,3 +360,39 @@
     </sensor>
   </gazebo>
+ <!-- hokuyo -->
+  <gazebo reference="laser_link">
+    <sensor type="gpu_ray" name="head_hokuyo_sensor">
+      <pose>0 0 0 0 0 0</pose>
+      <visualize>false</visualize>
+      <update_rate>40</update_rate>
+      <ray>
+        <scan>
+          <horizontal>
+            <samples>720</samples>
+            <resolution>1</resolution>
+            <min_angle>-1.570796</min_angle>
+            <max_angle>1.570796</max_angle>
+          </horizontal>
+        </scan>
+        <range>
+          <min>0.10</min>
+          <max>30.0</max>
+          <resolution>0.01</resolution>
+        </range>
+        <noise>
+          <type>gaussian</type>
+          <!-- Noise parameters based on published spec for Hokuyo laser
+               achieving "+-30mm" accuracy at range < 10m.  A mean of 0.0m and
+               stddev of 0.01m will put 99.7% of samples within 0.03m of the true
+               reading. -->
+          <mean>0.0</mean>
+          <stddev>0.01</stddev>
+        </noise>
+      </ray>
+      <plugin name="gazebo_ros_head_hokuyo_controller" filename="libgazebo_ros_gpu_laser.so">
+        <topicName>/laser/scan</topicName>
+        <frameName>laser_link</frameName>
+      </plugin>
+    </sensor>
+  </gazebo>
 </robot>

Commit message: Adjust wheel parameters

File: lk_rmc_description/urdf/model.xacro (robot description, xacro)
@@ -66,9 +66,9 @@
     <inertial>
       <origin xyz="0 0 0" rpy="0 0 0"/>
-      <mass value="5"/>
+      <mass value="2.637"/>
       <inertia
-        ixx="1.0" ixy="0.0" ixz="0.0"
-        iyy="1.0" iyz="0.0"
-        izz="1.0"/>
+        ixx=".02467" ixy="0.0" ixz="0.0"
+        iyy=".04411" iyz="0.0"
+        izz=".02467"/>
     </inertial>
   </link>
@@ -111,9 +111,9 @@
     <inertial>
       <origin xyz="0 0 0" rpy="0 0 0"/>
-      <mass value="5"/>
+      <mass value="2.637"/>
       <inertia
-        ixx="1.0" ixy="0.0" ixz="0.0"
-        iyy="1.0" iyz="0.0"
-        izz="1.0"/>
+        ixx=".02467" ixy="0.0" ixz="0.0"
+        iyy=".04411" iyz="0.0"
+        izz=".02467"/>
     </inertial>
   </link>
@@ -156,9 +156,9 @@
     <inertial>
       <origin xyz="0 0 0" rpy="0 0 0"/>
-      <mass value="5"/>
+      <mass value="2.637"/>
       <inertia
-        ixx="1.0" ixy="0.0" ixz="0.0"
-        iyy="1.0" iyz="0.0"
-        izz="1.0"/>
+        ixx=".02467" ixy="0.0" ixz="0.0"
+        iyy=".04411" iyz="0.0"
+        izz=".02467"/>
     </inertial>
   </link>
@@ -214,9 +214,9 @@
     <inertial>
       <origin xyz="0 0 0" rpy="0 0 0"/>
-      <mass value="5"/>
+      <mass value="2.637"/>
       <inertia
-        ixx="1.0" ixy="0.0" ixz="0.0"
-        iyy="1.0" iyz="0.0"
-        izz="1.0"/>
+        ixx=".02467" ixy="0.0" ixz="0.0"
+        iyy=".04411" iyz="0.0"
+        izz=".02467"/>
     </inertial>
   </link>
@@ -287,32 +287,32 @@
   </transmission>
   <!-- <gazebo reference="backRightWheel">
-    <mu1>0.1</mu1>
-    <mu2>0.1</mu2>
-    <kp>500000</kp>
-    <kd>10.0</kd>
+    <mu1>1.0</mu1>
+    <mu2>1.0</mu2>
+    <kp>10000000.0</kp>
+    <kd>1.0</kd>
     <minDepth>0.001</minDepth>
     <fdir1>1 0 0 </fdir1>
   </gazebo>
   <gazebo reference="backLeftWheel">
-    <mu1>0.1</mu1>
-    <mu2>0.1</mu2>
-    <kp>500000</kp>
-    <kd>10.0</kd>
+    <mu1>1.0</mu1>
+    <mu2>1.0</mu2>
+    <kp>10000000.0</kp>
+    <kd>1.0</kd>
     <minDepth>0.001</minDepth>
     <fdir1>1 0 0 </fdir1>
   </gazebo>
   <gazebo reference="frontRightWheel">
-    <mu1>0.1</mu1>
-    <mu2>0.1</mu2>
-    <kp>500000</kp>
-    <kd>10.0</kd>
+    <mu1>1.0</mu1>
+    <mu2>1.0</mu2>
+    <kp>10000000.0</kp>
+    <kd>1.0</kd>
     <minDepth>0.001</minDepth>
     <fdir1>1 0 0 </fdir1>
   </gazebo>
   <gazebo reference="frontLeftWheel">
-    <mu1>0.1</mu1>
-    <mu2>0.1</mu2>
-    <kp>500000</kp>
-    <kd>10.0</kd>
+    <mu1>1.0</mu1>
+    <mu2>1.0</mu2>
+    <kp>10000000.0</kp>
+    <kd>1.0</kd>
     <minDepth>0.001</minDepth>
     <fdir1>1 0 0 </fdir1>

Commit message: Set default gmapping parameters. Change laser link

File: lk_rmc_description/urdf/model.xacro (robot description, xacro)
@@ -237,5 +237,5 @@
     <parent link = "base_link"/>
     <child link="laser_link"/>
-    <origin xyz="0.385 0.0 0.235" rpy="0 0 0 "/>
+    <origin xyz="0.385 0.0 0.262" rpy="0 0 0 "/>
   </joint>
   <gazebo>
@@ -396,5 +396,5 @@
     <sensor type="gpu_ray" name="head_hokuyo_sensor">
       <pose>0 0 0 0 0 0</pose>
-      <visualize>false</visualize>
+      <visualize>true</visualize>
       <update_rate>40</update_rate>
       <ray>

Commit message: Fix merge problem (base link)

File: lk_rmc_description/urdf/model.xacro (robot description, xacro)
@@ -7,11 +7,4 @@
     <origin xyz="0.0 0.0 0.4" rpy="0 0 0 "/>
   </joint>
-  <link
-    name="base_link">
-  <!-- <link name="world"/> -->
-  <!-- <joint name="fixed" type="fixed">
-    <parent link="world"/>
-    <child link="base_link"/>
-  </joint> -->
 <!-- Main link that everything is based off of. base_link is default
 name that ros uses. Most properties generated through solidworks to URDF exporter-->

Commit message: Brandon 10 - Gazebo Setup (#12)
Initial  commit with folder structure and some files. Modified gitignore
Add Mission-Control package
Update readme
Initial copy from Sirdigsalot. Old robot model
Add files for gazebo package. Add empty world
Update package file names. TODO programmatic way
Added files. Rviz looks correct, gazebo doesnt
Fix some inertial properties. Working Gazebo

File: lk_rmc_description/urdf/model.xacro (robot description, xacro)
@@ -1,27 +1,12 @@
 <robot
   name="sirdigsalot">
-  <!-- <link name="world"/> -->
-  <!-- <joint name="fixed" type="fixed">
-    <parent link="world"/>
+  <link name="base_footprint"/>
+  <joint name="base_joint" type="fixed">
+    <parent link = "base_footprint"/>
     <child link="base_link"/>
-  </joint> -->
-<!-- Main link that everything is based off of. base_link is default
-name that ros uses. Most properties generated through solidworks to URDF exporter-->
+    <origin xyz="0.0 0.0 0.5" rpy="0 0 0 "/>
+  </joint>
   <link
     name="base_link">
-    <inertial>
-      <origin
-        xyz="0.0063713 -0.11708 0.0018811"
-        rpy="0 0 0" />
-      <mass
-        value="12.883" />
-      <inertia
-        ixx="0.27816"
-        ixy="-0.020687"
-        ixz="1.9963E-05"
-        iyy="0.59209"
-        iyz="3.0096E-05"
-        izz="0.60601" />
-    </inertial>
     <visual>
       <origin
@@ -47,22 +32,15 @@
       </geometry>
     </collision>
-  </link>
-  <!-- Wheel link for the front left wheel. Had to change to a cylinder to remove error-->
+    <inertial>
+      <origin xyz="0 0 -.25" rpy="0 0 0"/>
+      <mass value="12"/>
+      <inertia
+        ixx="1.0" ixy="0.0" ixz="0.0"
+        iyy="1.0" iyz="0.0"
+        izz="1.0"/>
+    </inertial>
+  </link>
   <link
     name="frontLeftWheel">
-    <inertial>
-      <origin
-        xyz="0 0 -0.0508"
-        rpy="0 0 0" />
-      <mass
-        value="7.4005" />
-      <inertia
-        ixx="0"
-        ixy="0"
-        ixz="0"
-        iyy="0"
-        iyz="0"
-        izz="0" />
-    </inertial>
     <visual>
       <origin
@@ -71,25 +49,28 @@
       <geometry>
           <cylinder length=".1016" radius=".1524"/>
-        <!-- <mesh
-          filename="package://lk_rmc_description/meshes/frontLeftWheel.STL" /> -->
-      </geometry>
-      <material
-        name="">
-        <color
-          rgba="0.79216 0.81961 0.93333 1" />
-      </material>
-    </visual>
-    <collision>
-      <origin
-        xyz="0 0 0"
-        rpy="0 0 0" />
-      <geometry>
-        <!-- <mesh
-          filename="package://lk_rmc_description/meshes/frontLeftWheel.STL" /> -->
-        <cylinder length=".1016" radius=".1524"/>
-      </geometry>
-    </collision>
-  </link>
-  <!--Joint for the front left wheel. Continious rotation link-->
+      </geometry>
+      <material
+        name="">
+        <color
+          rgba="0.79216 0.81961 0.93333 1" />
+      </material>
+    </visual>
+    <collision>
+      <origin
+        xyz="0 0 0"
+        rpy="0 0 0" />
+      <geometry>
+        <cylinder length=".1016" radius=".1524"/>
+      </geometry>
+    </collision>
+    <inertial>
+      <origin xyz="0 0 0" rpy="0 0 0"/>
+      <mass value="5"/>
+      <inertia
+        ixx="1.0" ixy="0.0" ixz="0.0"
+        iyy="1.0" iyz="0.0"
+        izz="1.0"/>
+    </inertial>
+  </link>
   <joint
     name="frontLeftWheelRotate"
@@ -107,43 +88,33 @@
   <link
     name="backLeftWheel">
-    <inertial>
-      <origin
-        xyz="-1.6653E-16 -1.9602E-16 -0.0508"
-        rpy="0 0 0" />
-      <mass
-        value="7.4005" />
-      <inertia
-        ixx="0"
-        ixy="0"
-        ixz="0"
-        iyy="0"
-        iyz="0"
-        izz="0" />
-    </inertial>
-    <visual>
-      <origin
-        xyz="0 0 0"
-        rpy="0 0 0" />
-      <geometry>
-        <!-- <mesh
-          filename="package://lk_rmc_description/meshes/backLeftWheel.STL" /> -->
-                  <cylinder length=".1016" radius=".1524"/>
-      </geometry>
-      <material
-        name="">
-        <color
-          rgba="0.79216 0.81961 0.93333 1" />
-      </material>
-    </visual>
-    <collision>
-      <origin
-        xyz="0 0 0"
-        rpy="0 0 0" />
-      <geometry>
-        <!-- <mesh
-          filename="package://lk_rmc_description/meshes/backLeftWheel.STL" /> -->
-                  <cylinder length=".1016" radius=".1524"/>
-      </geometry>
-    </collision>
+    <visual>
+      <origin
+        xyz="0 0 0"
+        rpy="0 0 0" />
+      <geometry>
+        <cylinder length=".1016" radius=".1524"/>
+      </geometry>
+      <material
+        name="">
+        <color
+          rgba="0.79216 0.81961 0.93333 1" />
+      </material>
+    </visual>
+    <collision>
+      <origin
+        xyz="0 0 0"
+        rpy="0 0 0" />
+      <geometry>
+        <cylinder length=".1016" radius=".1524"/>
+      </geometry>
+    </collision>
+    <inertial>
+      <origin xyz="0 0 0" rpy="0 0 0"/>
+      <mass value="5"/>
+      <inertia
+        ixx="1.0" ixy="0.0" ixz="0.0"
+        iyy="1.0" iyz="0.0"
+        izz="1.0"/>
+    </inertial>
   </link>
   <joint
@@ -162,43 +133,33 @@
   <link
     name="frontRightWheel">
-    <inertial>
-      <origin
-        xyz="0 0 0.0508"
-        rpy="0 0 0" />
-      <mass
-        value="7.4005" />
-      <inertia
-        ixx="0"
-        ixy="0"
-        ixz="0"
-        iyy="0"
-        iyz="0"
-        izz="0" />
-    </inertial>
-    <visual>
-      <origin
-        xyz="0 0 0"
-        rpy="0 0 0" />
-      <geometry>
-        <!-- <mesh
-          filename="package://lk_rmc_description/meshes/frontRightWheel.STL" /> -->
-                  <cylinder length=".1016" radius=".1524"/>
-      </geometry>
-      <material
-        name="">
-        <color
-          rgba="0.79216 0.81961 0.93333 1" />
-      </material>
-    </visual>
-    <collision>
-      <origin
-        xyz="0 0 0"
-        rpy="0 0 0" />
-      <geometry>
-        <!-- <mesh
-          filename="package://lk_rmc_description/meshes/frontRightWheel.STL" /> -->
-                  <cylinder length=".1016" radius=".1524"/>
-      </geometry>
-    </collision>
+    <visual>
+      <origin
+        xyz="0 0 0"
+        rpy="0 0 0" />
+      <geometry>
+        <cylinder length=".1016" radius=".1524"/>
+      </geometry>
+      <material
+        name="">
+        <color
+          rgba="0.79216 0.81961 0.93333 1" />
+      </material>
+    </visual>
+    <collision>
+      <origin
+        xyz="0 0 0"
+        rpy="0 0 0" />
+      <geometry>
+        <cylinder length=".1016" radius=".1524"/>
+      </geometry>
+    </collision>
+    <inertial>
+      <origin xyz="0 0 0" rpy="0 0 0"/>
+      <mass value="5"/>
+      <inertia
+        ixx="1.0" ixy="0.0" ixz="0.0"
+        iyy="1.0" iyz="0.0"
+        izz="1.0"/>
+    </inertial>
   </link>
   <joint
@@ -215,46 +176,4 @@
       xyz="0 0 1" />
   </joint>
-  <link
-    name="backRightWheel">
-    <inertial>
-      <origin
-        xyz="5.55111512312578E-17 0 0.0508"
-        rpy="0 0 0" />
-      <mass
-        value="7.40046273221895" />
-      <inertia
-        ixx="0"
-        ixy="0"
-        ixz="0"
-        iyy="0"
-        iyz="0"
-        izz="0" />
-    </inertial>
-    <visual>
-      <origin
-        xyz="0 0 0"
-        rpy="0 0 0" />
-      <geometry>
-        <!-- <mesh
-          filename="package://lk_rmc_description/meshes/backRightWheel.STL" /> -->
-                  <cylinder length=".1016" radius=".1524"/>
-      </geometry>
-      <material
-        name="">
-        <color
-          rgba="0.792156862745098 0.819607843137255 0.933333333333333 1" />
-      </material>
-    </visual>
-    <collision>
-      <origin
-        xyz="0 0 0"
-        rpy="0 0 0" />
-      <geometry>
-        <!-- <mesh
-          filename="package://lk_rmc_description/meshes/backRightWheel.STL" /> -->
-                  <cylinder length=".1016" radius=".1524"/>
-      </geometry>
-    </collision>
-  </link>
   <joint
     name="backRightWheelRotate"
@@ -270,292 +189,43 @@
       xyz="0 0 1" />
   </joint>
-  <!-- <link
-    name="depRightActuator">
-    <inertial>
-      <origin
-        xyz="-4.2562E-09 -0.020725 3.5813E-09"
-        rpy="0 0 0" />
-      <mass
-        value="0.088669" />
-      <inertia
-        ixx="0"
-        ixy="0"
-        ixz="0"
-        iyy="0"
-        iyz="0"
-        izz="0" />
-    </inertial>
-    <visual>
-      <origin
-        xyz="0 0 0"
-        rpy="0 0 0" />
-      <geometry>
-        <mesh
-          filename="package://lk_rmc_description/meshes/depRightActuator.STL" />
-      </geometry>
-      <material
-        name="">
-        <color
-          rgba="0.79216 0.81961 0.93333 1" />
-      </material>
-    </visual>
-    <collision>
-      <origin
-        xyz="0 0 0"
-        rpy="0 0 0" />
-      <geometry>
-        <mesh
-          filename="package://lk_rmc_description/meshes/depRightActuator.STL" />
-      </geometry>
-    </collision>
-  </link> -->
-  <!-- <joint
-    name="depRightExtend"
-    type="prismatic">
-    <origin
-      xyz="-0.11281 -0.18528 0"
-      rpy="-1.5708 0 0" />
-    <parent
-      link="base_link" />
-    <child
-      link="depRightActuator" />
-    <axis
-      xyz="0 -1 0" />
-    <limit
-      effort="0"
-      velocity="0" />
-  </joint>
-  <link
-    name="depConveyor">
-    <inertial>
-      <origin
-        xyz="0.28997 -6.0219E-05 0.15395"
-        rpy="0 0 0" />
-      <mass
-        value="22.501" />
-      <inertia
-        ixx="0.039859"
-        ixy="6.0953E-06"
-        ixz="0.047728"
-        iyy="0.097009"
-        iyz="-5.0904E-06"
-        izz="0.05715" />
-    </inertial>
-    <visual>
-      <origin
-        xyz="0 0 0"
-        rpy="0 0 0" />
-      <geometry>
-        <mesh
-          filename="package://lk_rmc_description/meshes/depConveyor.STL" />
-      </geometry>
-      <material
-        name="">
-        <color
-          rgba="0.79216 0.81961 0.93333 1" />
-      </material>
-    </visual>
-    <collision>
-      <origin
-        xyz="0 0 0"
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