Commit message: Added some files missing from Brandon-10.

File: lk_rmc_description/urdf/model.xacro (robot description, xacro)
@@ -1,4 +1,4 @@
-<robot
-  name="sirdigsalot">
+<robot name="sirdigsalot">
+  <!--Base Settings-->
   <link name="base_footprint"/>
   <joint name="base_joint" type="fixed">
@@ -7,6 +7,5 @@
     <origin xyz="0.0 0.0 0.5" rpy="0 0 0 "/>
   </joint>
-  <link
-    name="base_link">
+  <link name="base_link">
     <visual>
       <origin
@@ -41,6 +40,6 @@
     </inertial>
   </link>
-  <link
-    name="frontLeftWheel">
+  <!--Front Left Wheel Settings-->
+  <link name="backLeftWheel">
     <visual>
       <origin
@@ -50,8 +49,6 @@
           <cylinder length=".1016" radius=".1524"/>
       </geometry>
-      <material
-        name="">
-        <color
-          rgba="0.79216 0.81961 0.93333 1" />
+      <material name="">
+        <color rgba="0.79216 0.81961 0.93333 1" />
       </material>
     </visual>
@@ -66,50 +63,6 @@
     <inertial>
       <origin xyz="0 0 0" rpy="0 0 0"/>
-      <mass value="5"/>
-      <inertia
-        ixx="1.0" ixy="0.0" ixz="0.0"
-        iyy="1.0" iyz="0.0"
-        izz="1.0"/>
-    </inertial>
-  </link>
-  <joint
-    name="frontLeftWheelRotate"
-    type="continuous">
-    <origin
-      xyz="0.30464 0.23782 -0.28624"
-      rpy="1.5708 0.0022295 -1.3651E-19" />
-    <parent
-      link="base_link" />
-    <child
-      link="frontLeftWheel" />
-    <axis
-      xyz="0 0 1" />
-  </joint>
-  <link
-    name="backLeftWheel">
-    <visual>
-      <origin
-        xyz="0 0 0"
-        rpy="0 0 0" />
-      <geometry>
-        <cylinder length=".1016" radius=".1524"/>
-      </geometry>
-      <material
-        name="">
-        <color
-          rgba="0.79216 0.81961 0.93333 1" />
-      </material>
-    </visual>
-    <collision>
-      <origin
-        xyz="0 0 0"
-        rpy="0 0 0" />
-      <geometry>
-        <cylinder length=".1016" radius=".1524"/>
-      </geometry>
-    </collision>
-    <inertial>
-      <origin xyz="0 0 0" rpy="0 0 0"/>
-      <mass value="5"/>
+      <!--Old mass=5******************************************************-->
+      <mass value="2.37"/>
       <inertia
         ixx="1.0" ixy="0.0" ixz="0.0"
@@ -121,111 +74,16 @@
     name="backLeftWheelRotate"
     type="continuous">
-    <origin
-      xyz="-0.30496 0.23782 -0.28624"
-      rpy="1.5708 -0.71925 -3.6358E-15" />
-    <parent
-      link="base_link" />
-    <child
-      link="backLeftWheel" />
-    <axis
-      xyz="0 0 1" />
-  </joint>
-  <link
-    name="frontRightWheel">
-    <visual>
-      <origin
-        xyz="0 0 0"
-        rpy="0 0 0" />
-      <geometry>
-        <cylinder length=".1016" radius=".1524"/>
-      </geometry>
-      <material
-        name="">
-        <color
-          rgba="0.79216 0.81961 0.93333 1" />
-      </material>
-    </visual>
-    <collision>
-      <origin
-        xyz="0 0 0"
-        rpy="0 0 0" />
-      <geometry>
-        <cylinder length=".1016" radius=".1524"/>
-      </geometry>
-    </collision>
-    <inertial>
-      <origin xyz="0 0 0" rpy="0 0 0"/>
-      <mass value="5"/>
-      <inertia
-        ixx="1.0" ixy="0.0" ixz="0.0"
-        iyy="1.0" iyz="0.0"
-        izz="1.0"/>
-    </inertial>
-  </link>
-  <joint
-    name="frontRightWheelRotate"
-    type="continuous">
-    <origin
-      xyz="0.30464 -0.2416 -0.28624"
-      rpy="1.5708 -0.055957 3.4299E-18" />
-    <parent
-      link="base_link" />
-    <child
-      link="frontRightWheel" />
-    <axis
-      xyz="0 0 1" />
-  </joint>
-  <joint
-    name="backRightWheelRotate"
-    type="continuous">
-    <origin
-      xyz="-0.30496 -0.2416 -0.28624"
-      rpy="1.5708 0 0" />
-    <parent
-      link="base_link" />
-    <child
-      link="backRightWheel" />
-    <axis
-      xyz="0 0 1" />
-  </joint>
-  <link
-    name="backRightWheel">
-    <visual>
-      <origin
-        xyz="0 0 0"
-        rpy="0 0 0" />
-      <geometry>
-        <cylinder length=".1016" radius=".1524"/>
-      </geometry>
-      <material
-        name="">
-        <color
-          rgba="0.792156862745098 0.819607843137255 0.933333333333333 1" />
-      </material>
-    </visual>
-    <collision>
-      <origin
-        xyz="0 0 0"
-        rpy="0 0 0" />
-      <geometry>
-        <cylinder length=".1016" radius=".1524"/>
-      </geometry>
-    </collision>
-    <inertial>
-      <origin xyz="0 0 0" rpy="0 0 0"/>
-      <mass value="5"/>
-      <inertia
-        ixx="1.0" ixy="0.0" ixz="0.0"
-        iyy="1.0" iyz="0.0"
-        izz="1.0"/>
-    </inertial>
-  </link>
-  <gazebo>
-    <plugin name="gazebo_ros_control" filename="libgazebo_ros_control.so">
-      <robotNamespace></robotNamespace>
-      <!--robotParam>/robot_description</robotParam-->
-      <robotSimType>gazebo_ros_control/DefaultRobotHWSim</robotSimType>
-    </plugin>
-  </gazebo>
+    <!--
+    <origin
+      xyz="0.30464 0.23782 -0.28624"
+      rpy="1.5708 0.0022295 -1.3651E-19" />
+    -->
+    <origin
+      xyz="0.30464 0.2885 -0.28624"
+      rpy="1.5708 0.0022295 -1.3651E-19" />
+    <parent link="base_link" />
+    <child link="backLeftWheel" />
+    <axis xyz="0 0 1" />
+  </joint>
   <transmission name="backLeftWheelTrans" type="SimpleTransmission">
     <type>transmission_interface/SimpleTransmission</type>
@@ -238,4 +96,51 @@
     </joint>
   </transmission>
+  <!--Back Left Wheel Settings-->
+  <link name="frontLeftWheel">
+    <visual>
+      <origin
+        xyz="0 0 0"
+        rpy="0 0 0" />
+      <geometry>
+        <cylinder length=".1016" radius=".1524"/>
+      </geometry>
+      <material
+        name="">
+        <color
+          rgba="0.79216 0.81961 0.93333 1" />
+      </material>
+    </visual>
+    <collision>
+      <origin
+        xyz="0 0 0"
+        rpy="0 0 0" />
+      <geometry>
+        <cylinder length=".1016" radius=".1524"/>
+      </geometry>
+    </collision>
+    <inertial>
+      <origin xyz="0 0 0" rpy="0 0 0"/>
+      <mass value="2.37"/>
+      <inertia
+        ixx="1.0" ixy="0.0" ixz="0.0"
+        iyy="1.0" iyz="0.0"
+        izz="1.0"/>
+    </inertial>
+  </link>
+  <joint
+    name="frontLeftWheelRotate"
+    type="continuous">
+    <!--
+    <origin
+      xyz="-0.30496 0.23782 -0.28624"
+      rpy="1.5708 -0.71925 -3.6358E-15" />
+    -->
+    <origin
+      xyz="-0.30496 0.2885 -0.28624"
+      rpy="1.5708 -0.71925 -3.6358E-15" />
+    <parent link="base_link" />
+    <child link="frontLeftWheel" />
+    <axis xyz="0 0 1" />
+  </joint>
   <transmission name="frontLeftWheelTrans" type="SimpleTransmission">
     <type>transmission_interface/SimpleTransmission</type>
@@ -248,4 +153,52 @@
     </joint>
   </transmission>
+  <!--Front Right Wheel Settings-->
+  <link name="backRightWheel">
+    <visual>
+      <origin
+        xyz="0 0 0"
+        rpy="0 0 0" />
+      <geometry>
+        <cylinder length=".1016" radius=".1524"/>
+      </geometry>
+      <material
+        name="">
+        <color
+          rgba="0.79216 0.81961 0.93333 1" />
+      </material>
+    </visual>
+    <collision>
+      <origin
+        xyz="0 0 0"
+        rpy="0 0 0" />
+      <geometry>
+        <cylinder length=".1016" radius=".1524"/>
+      </geometry>
+    </collision>
+    <inertial>
+      <origin xyz="0 0 0" rpy="0 0 0"/>
+      <mass value="2.37"/>
+      <inertia
+        ixx="1.0" ixy="0.0" ixz="0.0"
+        iyy="1.0" iyz="0.0"
+        izz="1.0"/>
+    </inertial>
+  </link>
+  <joint
+    name="backRightWheelRotate"
+    type="continuous">
+    <!--
+    <origin
+      xyz="0.30464 -0.2416 -0.28624"
+      rpy="1.5708 -0.055957 3.4299E-18" />
+    -->
+    <!--r changes the yellow arrow side to point to the robot-->
+    <origin
+      xyz="0.30464 -0.2924 -0.28624"
+      rpy="-1.5708 -0.055957 3.4299E-18" />
+    <parent link="base_link" />
+    <child link="backRightWheel" />
+    <axis xyz="0 0 1" />
+  </joint>
   <transmission name="backRightWheelTrans" type="SimpleTransmission">
     <type>transmission_interface/SimpleTransmission</type>
@@ -258,4 +211,51 @@
     </joint>
   </transmission>
+  <!--Back Right Wheel Settings-->
+  <link name="frontRightWheel">
+    <visual>
+      <origin
+        xyz="0 0 0"
+        rpy="0 0 0" />
+      <geometry>
+        <cylinder length=".1016" radius=".1524"/>
+      </geometry>
+      <material
+        name="">
+        <color
+          rgba="0.792156862745098 0.819607843137255 0.933333333333333 1" />
+      </material>
+    </visual>
+    <collision>
+      <origin
+        xyz="0 0 0"
+        rpy="0 0 0" />
+      <geometry>
+        <cylinder length=".1016" radius=".1524"/>
+      </geometry>
+    </collision>
+    <inertial>
+      <origin xyz="0 0 0" rpy="0 0 0"/>
+      <mass value="2.37"/>
+      <inertia
+        ixx="1.0" ixy="0.0" ixz="0.0"
+        iyy="1.0" iyz="0.0"
+        izz="1.0"/>
+    </inertial>
+  </link>
+  <joint
+    name="frontRightWheelRotate"
+    type="continuous">
+    <!--
+    <origin
+      xyz="-0.30496 -0.2416 -0.28624"
+      rpy="1.5708 0 0" />
+    -->
+    <origin
+      xyz="-0.30496 -0.2924 -0.28624"
+      rpy="-1.5708 0 0" />
+    <parent link="base_link" />
+    <child link="frontRightWheel" />
+    <axis xyz="0 0 1" />
+  </joint>
   <transmission name="frontRightWheelTrans" type="SimpleTransmission">
     <type>transmission_interface/SimpleTransmission</type>
@@ -268,3 +268,52 @@
     </joint>
   </transmission>
+  <gazebo>
+    <plugin name="gazebo_ros_control" filename="libgazebo_ros_control.so">
+      <robotNamespace></robotNamespace>
+      <!--robotParam>/robot_description</robotParam-->
+      <robotSimType>gazebo_ros_control/DefaultRobotHWSim</robotSimType>
+    </plugin>
+  </gazebo>
+  <!--Laser Settings-->
+  <link name="laser_link"/>
+  <joint name="laser_link" type="fixed">
+    <parent link = "base_link"/>
+    <child link="laser_link"/>
+    <origin xyz="0.43 0.0 -0.2" rpy="0 0 0 "/>
+  </joint>
+  <gazebo reference="laser_link">
+    <sensor type="ray" name="head_hokuyo_sensor">
+      <pose>0 0 0 0 0 0</pose>
+      <visualize>true</visualize>
+      <update_rate>40</update_rate>
+      <ray>
+        <scan>
+          <horizontal>
+            <samples>720</samples>
+            <resolution>1</resolution>
+            <min_angle>-1.3</min_angle>
+            <max_angle>1.3</max_angle>
+          </horizontal>
+        </scan>
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
Commit message: Added Laser, IMU, Stereo Gazebo Sensors (#14)
* Initial  commit with folder structure and some files. Modified gitignore

* Add Mission-Control package

* Update readme

* Initial copy from Sirdigsalot. Old robot model

* Add files for gazebo package. Add empty world

* Update package file names. TODO programmatic way

* Added files. Rviz looks correct, gazebo doesnt

* Fix some inertial properties. Working Gazebo

* Add IMU & stereo sensor inputs from gazebo

* Added sensors and adjusted links to urdf

File: lk_rmc_description/urdf/model.xacro (robot description, xacro)
@@ -5,5 +5,5 @@
     <parent link = "base_footprint"/>
     <child link="base_link"/>
-    <origin xyz="0.0 0.0 0.5" rpy="0 0 0 "/>
+    <origin xyz="0.0 0.0 0.4" rpy="0 0 0 "/>
   </joint>
   <link
@@ -221,4 +221,22 @@
     </inertial>
   </link>
+  <link name="imu_link"/>
+  <joint name="imu_joint" type="fixed">
+    <parent link = "base_link"/>
+    <child link="imu_link"/>
+    <origin xyz="0.0 0.0 0.0" rpy="0 0 0 "/>
+  </joint>
+  <link name="camera_link"/>
+  <joint name="camera_link" type="fixed">
+    <parent link = "base_link"/>
+    <child link="camera_link"/>
+    <origin xyz="0.385 0.0 0.235" rpy="0 0 0 "/>
+  </joint>
+  <link name="laser_link"/>
+  <joint name="laser_link" type="fixed">
+    <parent link = "base_link"/>
+    <child link="laser_link"/>
+    <origin xyz="0.385 0.0 0.235" rpy="0 0 0 "/>
+  </joint>
   <gazebo>
     <plugin name="gazebo_ros_control" filename="libgazebo_ros_control.so">
@@ -268,3 +286,113 @@
     </joint>
   </transmission>
+  <gazebo reference="imu_link">
+    <gravity>true</gravity>
+    <sensor name="imu_sensor" type="imu">
+      <always_on>true</always_on>
+      <update_rate>100</update_rate>
+      <visualize>true</visualize>
+      <topic>__default_topic__</topic>
+      <plugin filename="libgazebo_ros_imu_sensor.so" name="imu_plugin">
+        <topicName>imu</topicName>
+        <bodyName>imu_link</bodyName>
+        <updateRateHZ>10.0</updateRateHZ>
+        <gaussianNoise>0.0</gaussianNoise>
+        <xyzOffset>0 0 0</xyzOffset>
+        <rpyOffset>0 0 0</rpyOffset>
+        <frameName>imu_link</frameName>
+      </plugin>
+      <pose>0 0 0 0 0 0</pose>
+    </sensor>
+  </gazebo>
+  <gazebo reference="camera_link">
+    <sensor type="multicamera" name="stereo_camera">
+      <update_rate>30.0</update_rate>
+      <camera name="left">
+        <horizontal_fov>1.3962634</horizontal_fov>
+        <image>
+          <width>800</width>
+          <height>800</height>
+          <format>R8G8B8</format>
+        </image>
+        <clip>
+          <near>0.02</near>
+          <far>300</far>
+        </clip>
+        <noise>
+          <type>gaussian</type>
+          <mean>0.0</mean>
+          <stddev>0.007</stddev>
+        </noise>
+      </camera>
+      <camera name="right">
+        <pose>0 -0.07 0 0 0 0</pose>
+        <horizontal_fov>1.3962634</horizontal_fov>
+        <image>
+          <width>800</width>
+          <height>800</height>
+          <format>R8G8B8</format>
+        </image>
+        <clip>
+          <near>0.02</near>
+          <far>300</far>
+        </clip>
+        <noise>
+          <type>gaussian</type>
+          <mean>0.0</mean>
+          <stddev>0.007</stddev>
+        </noise>
+      </camera>
+      <plugin name="stereo_camera_controller" filename="libgazebo_ros_multicamera.so">
+        <alwaysOn>true</alwaysOn>
+        <updateRate>0.0</updateRate>
+        <cameraName>multisense_sl/camera</cameraName>
+        <imageTopicName>image_raw</imageTopicName>
+        <cameraInfoTopicName>camera_info</cameraInfoTopicName>
+        <frameName>left_camera_optical_frame</frameName>
+        <!--<rightFrameName>right_camera_optical_frame</rightFrameName>-->
+        <hackBaseline>0.07</hackBaseline>
+        <distortionK1>0.0</distortionK1>
+        <distortionK2>0.0</distortionK2>
+        <distortionK3>0.0</distortionK3>
+        <distortionT1>0.0</distortionT1>
+        <distortionT2>0.0</distortionT2>
+      </plugin>
+    </sensor>
+  </gazebo>
+ <!-- hokuyo -->
+  <gazebo reference="laser_link">
+    <sensor type="gpu_ray" name="head_hokuyo_sensor">
+      <pose>0 0 0 0 0 0</pose>
+      <visualize>false</visualize>
+      <update_rate>40</update_rate>
+      <ray>
+        <scan>
+          <horizontal>
+            <samples>720</samples>
+            <resolution>1</resolution>
+            <min_angle>-1.570796</min_angle>
+            <max_angle>1.570796</max_angle>
+          </horizontal>
+        </scan>
+        <range>
+          <min>0.10</min>
+          <max>30.0</max>
+          <resolution>0.01</resolution>
+        </range>
+        <noise>
+          <type>gaussian</type>
+          <!-- Noise parameters based on published spec for Hokuyo laser
+               achieving "+-30mm" accuracy at range < 10m.  A mean of 0.0m and
+               stddev of 0.01m will put 99.7% of samples within 0.03m of the true
+               reading. -->
+          <mean>0.0</mean>
+          <stddev>0.01</stddev>
+        </noise>
+      </ray>
+      <plugin name="gazebo_ros_head_hokuyo_controller" filename="libgazebo_ros_gpu_laser.so">
+        <topicName>/laser/scan</topicName>
+        <frameName>laser_link</frameName>
+      </plugin>
+    </sensor>
+  </gazebo>
 </robot>
